Commit message: Full project first commit

File: src/phoxi_camera/urdf/PhoXi3Dscanner_macro.xacro (robot description, xacro)
@@ -11,5 +11,5 @@
           <mesh filename="package://phoxi_camera/meshes/visual/PhoXi3DScannerS.dae" scale = "0.01 0.01 0.01"/>
         </geometry>
-      <origin xyz="0 0 0" rpy="${pi/2} 0 ${-pi}"/>
+        <origin xyz="0 0 0" rpy="${pi/2} 0 ${-pi}"/>
       </visual>
       <collision>
@@ -18,4 +18,5 @@
           <mesh filename="package://phoxi_camera/meshes/collision/PhoXi3DScannerSCollision.stl" scale = "0.001 0.001 0.001"/>
         </geometry>
+        <origin xyz="0 0 0" rpy="${pi/2} 0 ${-pi}"/>
         <xacro:collision_colour />
       </collision>
@@ -30,6 +31,6 @@
     <joint name="camera_support_to_PhoXi3Dscanner_joint" type="fixed">
       <origin xyz="0.555 -0.384 1.3815" rpy="0 0 0"/>
+      <child link="PhoXi3Dscanner"/>
       <parent link="ConveyorAndSupportComponents"/>
-      <child link="PhoXi3Dscanner"/>
     </joint>
     <!-- Sensor joint when using the "CameraSpace" coordinate system ***NEEDS ADJUSTMENTS*** -->
@@ -42,6 +43,6 @@
     <joint name="PhoXi3Dscanner_to_PhoXi3Dscanner_sensor_MarkerSpace_joint" type="fixed">
       <origin xyz="0.135 -0.0378 -0.5425" rpy="0 0 0" />
+      <child link="PhoXi3Dscanner_sensor"/>
       <parent link="PhoXi3Dscanner"/>
-      <child link="PhoXi3Dscanner_sensor"/>
     </joint>
     <!-- end of joint list -->

File: src/pick_and_place_env/urdf/Fixed_parts_macro.xacro (robot description, xacro)
@@ -50,12 +50,12 @@
       <origin xyz="0 0 0" rpy="0 0 0"/>
       <axis xyz="0 0 1"/>
+      <child link="SafetyAndControllerComponents"/>
       <parent link="RoomComponents"/>
-      <child link="SafetyAndControllerComponents"/>
     </joint>
     <joint name="Room_to_ConveyorAndSupport_joint" type="fixed">
       <origin xyz="0 0 0" rpy="0 0 0"/>
       <axis xyz="0 0 1"/>
+      <child link="ConveyorAndSupportComponents"/>
       <parent link="RoomComponents"/>
-      <child link="ConveyorAndSupportComponents"/>
     </joint>
     <!-- end of joint list -->
